File: pcb/X-PAD/X-PAD.kicad_sch (KiCad schematic)
At the start: 74 parts, among them Q1 BSS138, SW1 SW_MEC_5G, SW10 SW_MEC_5G, SW11 SW_MEC_5G, SW12 SW_MEC_5G, SW13 SW_MEC_5G, SW14 SW_MEC_5G, SW15 SW_MEC_5G, SW16 SW_MEC_5G, SW2 SW_MEC_5G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

Commit message: applied
Other:
- company: Cyber Link -- A Hack Club -> (none)
- title: HackPad V3 -> X-PAD
Changed lines of the file:
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@@
 	(paper "A4")
 	(title_block
-		(title "HackPad V3")
+		(title "X-PAD")
 		(date "2025-05-07")
 		(rev "V0.2")
-		(company "Cyber Link -- A Hack Club")
 		(comment 1 "A simple (not so simple) macropad with as much as features that I can do for my first build")
 		(comment 2 "2 Rotary Encoders, a 0.91\" OLED, and more!")
